File: pcb/c64a/c64a.kicad_pcb (KiCad board)
At the start: 2 copper layers, 375 x 107 mm, 146 parts, among them J1 Conn_01x20_Male, SW1 1, SW10 3, SW11 W, SW12 A, SW13 L-SHIFT, SW14 Z, SW15 S, SW16 E, SW17 4, SW18 5, SW19 R, SW2 L-ARROW, SW20 D, SW21 X, SW22 C, SW23 F, SW24 T, SW25 6, SW26 7, SW27 Y, SW28 G, SW29 V, SW3 CTRL, SW30 B, SW31 H, SW32 U, SW33 8, SW34 9, SW35 I, SW36 J, SW37 N, SW38 M, SW39 K, SW4 RUN / STOP, SW40 O, SW41 0, SW42 +, SW43 P, SW44 L, SW45 ,, SW46 ., SW47 :, SW48 @, SW49 -, SW5 SPACE, SW50 POUND, SW51 *, SW52 ;, SW53 /, SW54 R-SHIFT, SW55 =, SW56 UP-ARROW, SW57 HOME, SW58 RESTORE, SW59 DEL, SW6 COMMODORE, SW60 RETURN, SW61 LEFT-RIGHT, SW62 UP-DOWN, SW63 F1, SW64 F3, SW65 F5, SW66 F7, SW7 Q, SW8 2, SW9 SHIFT-LOCK

Commit message: Switches changed to 5 pin
Parts:
- removed D57: D_Small, Diode_SMD:D_SOD-123
- removed H10, H11, H12, H13, H14, H7, H8, H9: M_HOLE, MountingHole:MountingHole_2.2mm_M2
- SW1, SW10, SW11, SW12, SW13, SW14, SW15, SW16, SW17, SW18, SW19, SW2, SW20, SW21, SW22, SW23, SW24, SW25, SW26, SW27, SW28, SW29, SW3, SW30, SW31, SW32, SW33, SW34, SW35, SW36, SW37, SW38, SW39, SW4, SW40, SW41, SW42, SW43, SW44, SW45, SW46, SW47, SW48, SW49, SW5, SW50, SW51, SW52, SW53, SW54, SW55, SW56, SW57, SW58, SW59, SW6, SW60, SW61, SW62, SW63, SW64, SW65, SW66, SW7, SW8, SW9: footprint Switch_Keyboard_Cherry_MX:SW_Cherry_MX_Plate_1.00u -> Button_Switch_Keyboard:SW_Cherry_MX_1.00u_PCB
- moved SW25 5.59 mm to (104.8, -103.8)
- moved SW26 5.59 mm to (123.9, -103.8)
- moved SW32 5.59 mm to (133.3, -84.7)
- moved SW33 5.59 mm to (142.9, -103.8)
- moved SW34 5.59 mm to (162.0, -103.8)
- moved SW40 5.59 mm to (171.4, -84.7)
- moved SW41 5.59 mm to (181.0, -103.8)
- moved SW42 5.59 mm to (200.1, -103.8)
- moved SW43 5.59 mm to (190.5, -84.7)
- moved SW44 5.59 mm to (176.1, -65.6)
- moved SW47 5.59 mm to (195.2, -65.6)
- moved SW55 5.59 mm to (233.4, -65.6)
- moved SW58 5.59 mm to (266.8, -84.7)
- moved SW59 5.59 mm to (276.3, -103.8)
- moved SW60 5.59 mm to (261.9, -65.6)
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Connections:
- SW1 pad 1: Net-(D1-Pad2) -> R0
- SW1 pad 2: R0 -> Net-(D1-Pad2)
- SW10 pad 1: Net-(D9-Pad2) -> R0
- SW10 pad 2: R0 -> Net-(D9-Pad2)
- SW11 pad 1: Net-(D10-Pad2) -> R1
- SW11 pad 2: R1 -> Net-(D10-Pad2)
- SW12 pad 1: Net-(D11-Pad2) -> R2
- SW12 pad 2: R2 -> Net-(D11-Pad2)
- SW13 pad 1: Net-(D12-Pad2) -> R3
- SW13 pad 2: R3 -> Net-(D12-Pad2)
- SW14 pad 1: Net-(D13-Pad2) -> R4
- SW14 pad 2: R4 -> Net-(D13-Pad2)
- SW15 pad 1: Net-(D14-Pad2) -> R5
- SW15 pad 2: R5 -> Net-(D14-Pad2)
- SW16 pad 1: Net-(D15-Pad2) -> R6
- SW16 pad 2: R6 -> Net-(D15-Pad2)
- SW17 pad 1: Net-(D16-Pad2) -> R7
- SW17 pad 2: R7 -> Net-(D16-Pad2)
- SW18 pad 1: Net-(D17-Pad2) -> R0
- SW18 pad 2: R0 -> Net-(D17-Pad2)
- SW19 pad 1: Net-(D18-Pad2) -> R1
- SW19 pad 2: R1 -> Net-(D18-Pad2)
- SW2 pad 1: Net-(D2-Pad2) -> R1
- SW2 pad 2: R1 -> Net-(D2-Pad2)
- SW20 pad 1: Net-(D19-Pad2) -> R2
- SW20 pad 2: R2 -> Net-(D19-Pad2)
- SW21 pad 1: Net-(D20-Pad2) -> R3
- SW21 pad 2: R3 -> Net-(D20-Pad2)
- SW22 pad 1: Net-(D21-Pad2) -> R4
- SW22 pad 2: R4 -> Net-(D21-Pad2)
- SW23 pad 1: Net-(D22-Pad2) -> R5
- SW23 pad 2: R5 -> Net-(D22-Pad2)
- SW24 pad 1: Net-(D23-Pad2) -> R6
- SW24 pad 2: R6 -> Net-(D23-Pad2)
- SW25 pad 1: Net-(D24-Pad2) -> R7
- SW25 pad 2: R7 -> Net-(D24-Pad2)
- SW26 pad 1: Net-(D25-Pad2) -> R0
- SW26 pad 2: R0 -> Net-(D25-Pad2)
- SW27 pad 1: Net-(D26-Pad2) -> R1
- SW27 pad 2: R1 -> Net-(D26-Pad2)
- SW28 pad 1: Net-(D27-Pad2) -> R2
- SW28 pad 2: R2 -> Net-(D27-Pad2)
- SW29 pad 1: Net-(D28-Pad2) -> R3
- SW29 pad 2: R3 -> Net-(D28-Pad2)
- SW3 pad 1: Net-(D3-Pad2) -> R2
- SW3 pad 2: R2 -> Net-(D3-Pad2)
- SW30 pad 1: Net-(D29-Pad2) -> R4
- SW30 pad 2: R4 -> Net-(D29-Pad2)
- SW31 pad 1: Net-(D30-Pad2) -> R5
- SW31 pad 2: R5 -> Net-(D30-Pad2)
- SW32 pad 1: Net-(D31-Pad2) -> R6
- SW32 pad 2: R6 -> Net-(D31-Pad2)
- SW33 pad 1: Net-(D32-Pad2) -> R7
- SW33 pad 2: R7 -> Net-(D32-Pad2)
- SW34 pad 1: Net-(D33-Pad2) -> R0
- SW34 pad 2: R0 -> Net-(D33-Pad2)
- SW35 pad 1: Net-(D34-Pad2) -> R1
- SW35 pad 2: R1 -> Net-(D34-Pad2)
- SW36 pad 1: Net-(D35-Pad2) -> R2
- SW36 pad 2: R2 -> Net-(D35-Pad2)
- SW37 pad 1: Net-(D36-Pad2) -> R3
- SW37 pad 2: R3 -> Net-(D36-Pad2)
- SW38 pad 1: Net-(D37-Pad2) -> R4
- SW38 pad 2: R4 -> Net-(D37-Pad2)
- SW39 pad 1: Net-(D38-Pad2) -> R5
- SW39 pad 2: R5 -> Net-(D38-Pad2)
- SW4 pad 1: Net-(D4-Pad2) -> R3
- SW4 pad 2: R3 -> Net-(D4-Pad2)
- SW40 pad 1: Net-(D39-Pad2) -> R6
- SW40 pad 2: R6 -> Net-(D39-Pad2)
- SW41 pad 1: Net-(D40-Pad2) -> R7
- SW41 pad 2: R7 -> Net-(D40-Pad2)
- SW42 pad 1: Net-(D41-Pad2) -> R0
- SW42 pad 2: R0 -> Net-(D41-Pad2)
- SW43 pad 1: Net-(D42-Pad2) -> R1
- SW43 pad 2: R1 -> Net-(D42-Pad2)
- SW44 pad 1: Net-(D43-Pad2) -> R2
- SW44 pad 2: R2 -> Net-(D43-Pad2)
- SW45 pad 1: Net-(D44-Pad2) -> R3
- SW45 pad 2: R3 -> Net-(D44-Pad2)
- SW46 pad 1: Net-(D45-Pad2) -> R4
- SW46 pad 2: R4 -> Net-(D45-Pad2)
- SW47 pad 1: Net-(D46-Pad2) -> R5
- SW47 pad 2: R5 -> Net-(D46-Pad2)
- SW48 pad 1: Net-(D47-Pad2) -> R6
- SW48 pad 2: R6 -> Net-(D47-Pad2)
- SW49 pad 1: Net-(D48-Pad2) -> R7
- SW49 pad 2: R7 -> Net-(D48-Pad2)
- SW5 pad 1: Net-(D5-Pad2) -> R4
- SW5 pad 2: R4 -> Net-(D5-Pad2)
- SW50 pad 1: Net-(D49-Pad2) -> R0
- SW50 pad 2: R0 -> Net-(D49-Pad2)
- SW51 pad 1: Net-(D50-Pad2) -> R1
- SW51 pad 2: R1 -> Net-(D50-Pad2)
- SW52 pad 1: Net-(D51-Pad2) -> R2
- SW52 pad 2: R2 -> Net-(D51-Pad2)
- SW53 pad 1: Net-(D52-Pad2) -> R3
- SW53 pad 2: R3 -> Net-(D52-Pad2)
- SW54 pad 1: Net-(D53-Pad2) -> R4
- SW54 pad 2: R4 -> Net-(D53-Pad2)
- SW55 pad 1: Net-(D54-Pad2) -> R5
- SW55 pad 2: R5 -> Net-(D54-Pad2)
- SW56 pad 1: Net-(D55-Pad2) -> R6
- SW56 pad 2: R6 -> Net-(D55-Pad2)
- SW57 pad 1: Net-(D56-Pad2) -> R7
- SW57 pad 2: R7 -> Net-(D56-Pad2)
- SW58 pad 1: Net-(D57-Pad2) -> R8
- SW58 pad 2: R8 -> I
- SW59 pad 1: Net-(D58-Pad2) -> R0
- SW59 pad 2: R0 -> Net-(D58-Pad2)
- SW6 pad 1: Net-(D6-Pad2) -> R5
- SW6 pad 2: R5 -> Net-(D6-Pad2)
- SW60 pad 1: Net-(D59-Pad2) -> R1
- SW60 pad 2: R1 -> Net-(D59-Pad2)
- SW61 pad 1: Net-(D60-Pad2) -> R2
- SW61 pad 2: R2 -> Net-(D60-Pad2)
- SW62 pad 1: Net-(D61-Pad2) -> R3
- SW62 pad 2: R3 -> Net-(D61-Pad2)
- SW63 pad 1: Net-(D62-Pad2) -> R4
- SW63 pad 2: R4 -> Net-(D62-Pad2)
- SW64 pad 1: Net-(D63-Pad2) -> R5
- SW64 pad 2: R5 -> Net-(D63-Pad2)
- SW65 pad 1: Net-(D64-Pad2) -> R6
- SW65 pad 2: R6 -> Net-(D64-Pad2)
- SW66 pad 1: Net-(D65-Pad2) -> R7
- SW66 pad 2: R7 -> Net-(D65-Pad2)
- SW7 pad 1: Net-(D7-Pad2) -> R6
- SW7 pad 2: R6 -> Net-(D7-Pad2)
- SW8 pad 1: Net-(D8-Pad2) -> R7
- SW8 pad 2: R7 -> Net-(D8-Pad2)
- SW9 pad 1: Net-(D12-Pad2) -> R3
- SW9 pad 2: R3 -> Net-(D12-Pad2)
Routing:
- net I: track 20.8 -> 36.5 mm
- net Net-(D57-Pad2): track 12.4 -> 0.00 mm
- net A: track 572.8 -> 568.0 mm
- net Net-(D59-Pad2): track 8.28 -> 13.1 mm
- net Net-(D12-Pad2): track 26.4 -> 31.2 mm
- net Net-(D19-Pad2): track 7.92 -> 9.83 mm
- net Net-(D22-Pad2): track 7.96 -> 9.72 mm
- net Net-(D16-Pad2): track 8.03 -> 9.67 mm
- net Net-(D27-Pad2): track 7.97 -> 9.61 mm
- net Net-(D49-Pad2): track 7.75 -> 9.34 mm
- net Net-(D54-Pad2): track 8.05 -> 9.61 mm
- net Net-(D43-Pad2): track 8.12 -> 9.62 mm
- net Net-(D51-Pad2): track 8.19 -> 9.66 mm
- net Net-(D9-Pad2): track 8.03 -> 9.44 mm
- net Net-(D8-Pad2): track 7.99 -> 9.40 mm
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
Commit message: Mount cover + pcb fixes
Parts:
- J1: footprint Connector_PinHeader_1.00mm:PinHeader_1x20_P1.00mm_Horizontal -> Connector_PinHeader_1.27mm:PinHeader_1x20_P1.27mm_Horizontal
- moved H2 137.2 mm to (29.6, 15.0)
- moved H4 128.7 mm to (17.5, 15.2)
- moved H5 119.1 mm to (25.8, 15.2)
- moved H1 110.8 mm to (21.8, 15.2)
- moved SW54 8.41 mm to (232.3, -46.8)
- moved D53 7.12 mm to (220.2, -46.5)
- moved J1 6.03 mm to (284.1, -93.6)
- moved SW62 1.20 mm to (270.3, -46.8)
- moved SW60 1.11 mm to (260.8, -65.8)
- moved SW61 1.11 mm to (251.3, -46.8)
- moved SW52 1.11 mm to (213.3, -65.8)
- moved SW55 1.11 mm to (232.3, -65.8)
- moved H6 1.06 mm to (258.4, -60.8)
- moved SW53 1.01 mm to (203.8, -46.8)
- moved SW47 0.91 mm to (194.3, -65.8)
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Routing:
- net R2: track 724.1 -> 713.7 mm
- net I: track 36.5 -> 29.3 mm
- net G: track 170.3 -> 177.4 mm
- net R0: track 507.9 -> 501.4 mm
- net R8: track 33.7 -> 27.6 mm
- net C: track 345.2 -> 349.3 mm
- net D: track 304.1 -> 308.2 mm
- net F: track 222.7 -> 226.8 mm
- net H: track 198.7 -> 195.1 mm
- net R5: track 421.2 -> 417.8 mm
- net R3: track 489.9 -> 486.7 mm
- net E: track 265.2 -> 268.0 mm
- net R6: track 382.1 -> 379.4 mm
- net Net-(D59-Pad2): track 13.1 -> 15.5 mm
- net Net-(D32-Pad2): track 7.95 -> 9.84 mm
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Other:
- board size 375 x 107 mm -> 375 x 108 mm

Commit message: Outline fixes
Routing:
- net R0: track 501.4 -> 490.7 mm
- net R2: track 713.7 -> 710.1 mm
Other:
- outline, holes or cut-outs redrawn

Commit message: Fixing spacing issues
Parts:
- removed H1, H2, H4, H5: M_HOLE, MountingHole:MountingHole_2.2mm_M2
- J1: footprint Connector_PinHeader_1.27mm:PinHeader_1x20_P1.27mm_Horizontal -> Connector_PinHeader_2.54mm:PinHeader_1x20_P2.54mm_Horizontal
- moved J1 19.0 mm to (265.6, -89.5)
- moved D3 8.33 mm to (-19.3, -84.8)
- moved D64 7.86 mm to (306.3, -61.5)
- moved D65 6.34 mm to (310.7, -50.2)
- moved D63 5.02 mm to (309.4, -84.8)
- moved SW66 4.75 mm to (322.1, -46.7)
- moved SW58 4.75 mm to (270.6, -84.8)
- moved SW54 4.75 mm to (227.6, -46.8)
- moved SW3 4.75 mm to (-4.88, -84.8)
- moved SW63 4.75 mm to (322.1, -103.8)
- moved SW65 4.75 mm to (322.1, -65.8)
- moved SW64 4.65 mm to (322.2, -84.8)
- moved SW13 4.65 mm to (9.17, -46.8)
- moved D12 3.96 mm to (-2.47, -46.4)
- moved D62 3.70 mm to (312.1, -98.7)
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Routing:
- net R8: track 27.6 -> 4.64 mm
- net I: track 29.3 -> 7.71 mm
- net R3: track 486.7 -> 470.6 mm
- net H: track 195.1 -> 179.2 mm
- net R2: track 710.1 -> 696.1 mm
- net R1: track 363.4 -> 352.1 mm
- net A: track 567.8 -> 559.1 mm
- net B: track 390.2 -> 398.5 mm
- net R6: track 379.4 -> 371.9 mm
- net R0: track 490.7 -> 484.8 mm
- net Net-(D65-Pad2): track 4.61 -> 8.84 mm
- net Net-(D64-Pad2): track 4.62 -> 8.57 mm
- net Net-(D3-Pad2): track 4.71 -> 8.42 mm
- net C: track 349.3 -> 352.5 mm
- net R4: track 364.9 -> 362.1 mm
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Other:
- board size 375 x 108 mm -> 357 x 107.5 mm
